File: Modulo_Regulador/Modulo_Regulador.kicad_sch (KiCad schematic)
At the start: 9 parts, among them U2 AMS1117-5.0

Commit message: Some changes in arduino board.
Parts:
- renumbered C9 to C10, C10 to C11, C11 to C12, C7 to C8, C8 to C9, R3 to R4
Changed lines of the file:
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@@
 		(dnp no)
 		(fields_autoplaced yes)
-		(property "Reference" "C9"
+		(property "Reference" "C10"
 			(at 148.59 87.6362 0)
 			(effects
@@
 			(project "Modulo_Regulador"
 				(path "/b1260de1-9c48-4b08-a759-f31e40d6183e/9c3fd946-361f-4818-a9de-72eecbd2c7bd"
-					(reference "C9")
+					(reference "C10")
 					(unit 1)
 				)
@@
 		(dnp no)
 		(fields_autoplaced yes)
-		(property "Reference" "R3"
+		(property "Reference" "R4"
 			(at 166.37 101.6 90)
 			(effects
@@
 			(project "Modulo_Regulador"
 				(path "/b1260de1-9c48-4b08-a759-f31e40d6183e/9c3fd946-361f-4818-a9de-72eecbd2c7bd"
-					(reference "R3")
+					(reference "R4")
 					(unit 1)
 				)
@@
 		(dnp no)
 		(fields_autoplaced yes)
-		(property "Reference" "C11"
+		(property "Reference" "C12"
 			(at 200.66 87.6362 0)
 			(effects
@@
 			(project "Modulo_Regulador"
 				(path "/b1260de1-9c48-4b08-a759-f31e40d6183e/9c3fd946-361f-4818-a9de-72eecbd2c7bd"
-					(reference "C11")
+					(reference "C12")
 					(unit 1)
 				)
@@
 		(dnp no)
 		(fields_autoplaced yes)
-		(property "Reference" "C7"
+		(property "Reference" "C8"
 			(at 119.38 87.6362 0)
 			(effects
@@
 			(project "Modulo_Regulador"
 				(path "/b1260de1-9c48-4b08-a759-f31e40d6183e/9c3fd946-361f-4818-a9de-72eecbd2c7bd"
-					(reference "C7")
+					(reference "C8")
 					(unit 1)
 				)
@@
 		(on_board yes)
 		(dnp no)
-		(property "Reference" "C10"
+		(property "Reference" "C11"
 			(at 182.88 87.6362 0)
 			(effects
@@
 			(project "Modulo_Regulador"
 				(path "/b1260de1-9c48-4b08-a759-f31e40d6183e/9c3fd946-361f-4818-a9de-72eecbd2c7bd"
-					(reference "C10")
+					(reference "C11")
 					(unit 1)
 				)
@@
 		(dnp no)
 		(fields_autoplaced yes)
-		(property "Reference" "C8"
+		(property "Reference" "C9"
 			(at 134.62 87.6362 0)
 			(effects
@@
 			(project "Modulo_Regulador"
 				(path "/b1260de1-9c48-4b08-a759-f31e40d6183e/9c3fd946-361f-4818-a9de-72eecbd2c7bd"
-					(reference "C8")
-					(unit 1)
-				)
+					(reference "C9")
+					(unit 1)
+				)

Commit message: First version from PCB schematic.
Connections:
- net 12V renamed +12V
- net 5V renamed +5V
Changed lines of the file:
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@@
 		)
 	)
-	(hierarchical_label "5V"
+	(hierarchical_label "+5V"
 		(shape input)
 		(at 172.72 107.95 0)
@@
 		)
 	)
-	(hierarchical_label "5V"
+	(hierarchical_label "+5V"
 		(shape input)
 		(at 208.28 83.82 0)
@@
 		)
 	)
-	(hierarchical_label "12V"
+	(hierarchical_label "+12V"
 		(shape input)
 		(at 132.08 77.47 90)
