File: Arduino/Arduino.kicad_pcb (KiCad board)
At the start: 2 copper layers, 98 x 116.3 mm, 120 parts, among them J1 Barrel_Jack_Switch, J10 I2C, J11 Digital, J12 Digital, J13 USB_C_Receptacle_USB2.0, J14 USB_B, J15 Conn_01x04, J16 Screw_Terminal_01x12, J17 Conn_01x01, J18 Conn_01x01, J19 Conn_01x01, J2 Vcc, J20 Pin, J21 Bt_ext, J22 Pin, J23 Bt_ext, J24 Pin, J25 Pin, J26 Conn_01x01, J3 ICSP, J4 Conn_01x03, J5 Servo, J6 Conn_01x01, J7 Conn_01x01, J8 Power, J9 Digital, K1 G5LE-1, K2 G5LE-1, K3 G5LE-1, K4 G5LE-1, Q1 SS8050, Q2 SS8050, Q3 SS8050, Q4 SS8050, Q5 SS8050, Q6 SS8050, SW1 Reset, SW2 Button, SW3 Button, U1 ATmega328P-P, U2 AMS1117-5.0, U3 CH340G, Y1 16MHz, Y2 12Mhz

Commit message: Final adjustments in arduino board
Routing:
- added copper zone on B.Cu, net (none)
- added copper zone on F.Cu, net (none)
- added copper zone on F.Cu, net GND
Changed lines of the file:
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@@
+	)
+	(zone
+		(net 0)
+		(net_name "")
+		(layer "F.Cu")
+		(hatch edge 0.5)
+		(priority 4)
+		(connect_pads yes
+			(clearance 0.5)
+		)
+		(min_thickness 0.25)
+		(filled_areas_thickness no)
+		(fill yes
+			(thermal_gap 0.5)
+			(thermal_bridge_width 0.5)
+			(island_removal_mode 1)
+			(island_area_min 10)
+		)
+		(polygon
+			(pts
+				(xy 121.55 114.75) (xy 128.7 114.75) (xy 128.75 121.05) (xy 121.55 121.05)
+			)
+		)
 	)
 	(zone
@@
 				(xy 113.8 111.5) (xy 135.4 111.5) (xy 135.4 124.5) (xy 101.3 124.5) (xy 101.3 140.4) (xy 108.6 147.9)
 				(xy 163.15 147.9) (xy 166.8 143.2) (xy 168.55 144.35) (xy 168.55 149.5) (xy 99.2 149.55) (xy 99.2 63.1)
+			)
+		)
+	)
+	(zone
+		(net 6)
+		(net_name "GND")
+		(layer "F.Cu")
+		(hatch edge 0.5)
+		(priority 5)
+		(connect_pads
+			(clearance 0.5)
+		)
+		(min_thickness 0.25)
+		(filled_areas_thickness no)
+		(fill yes
+			(thermal_gap 0.5)
+			(thermal_bridge_width 0.5)
+		)
+		(polygon
+			(pts
+				(xy 121.55 114.75) (xy 128.7 114.75) (xy 128.75 121.05) (xy 121.55 121.05)
+			)
+		)
+	)
+	(zone
+		(net 0)
+		(net_name "")
+		(layers "F.Cu" "B.Cu")
+		(hatch edge 0.5)
+		(connect_pads
+			(clearance 0.5)
+		)
+		(min_thickness 0.25)
+		(filled_areas_thickness no)
+		(fill yes
+			(thermal_gap 0.5)
+			(thermal_bridge_width 0.5)
+			(island_removal_mode 1)
+			(island_area_min 10)
+		)
+		(polygon
+			(pts
+				(xy 121.55 114.75) (xy 128.7 114.75) (xy 128.75 121.05) (xy 121.55 121.05)
+			)
+		)
+	)
+	(zone
+		(net 0)
+		(net_name "")
+		(layers "F.Cu" "B.Cu")
+		(hatch edge 0.5)
+		(priority 3)
+		(connect_pads yes
+			(clearance 0.5)
+		)
+		(min_thickness 0.25)
+		(filled_areas_thickness no)
+		(fill yes
+			(thermal_gap 0.5)
+			(thermal_bridge_width 0.5)
+			(island_removal_mode 1)
+			(island_area_min 10)
+		)
+		(polygon
+			(pts
+				(xy 121.55 114.75) (xy 128.7 114.75) (xy 128.75 121.05) (xy 121.55 121.05)
 			)
 		)
@@
 			"07ee8929-e75e-40cd-b2d9-8468161b6583" "0c13ebb7-e01a-474d-9311-d6fb85d33555"
 			"147a42f0-78ac-4d25-9a81-34987b4c8259" "17dd3f51-9127-42c8-9c3d-ad9293a84a7a"
-			"189e168f-b7a0-484c-aa2a-fdb9d9e916c6" "20235f43-cf96-4218-aa84-5a156a011ff2"
-			"26c525f2-d4d9-4653-8977-4d813e08275d" "29dd66b1-5e01-40b9-8e29-19c8a0c273a8"
-			"2c4f203c-5b0c-4867-8517-6ca5922d05ff" "2cb49122-9564-4c5b-856a-4b720769080a"
-			"301259ed-6e02-41d2-bbbf-7d9d5a8ac4dd" "3c5fac19-14d4-4494-9de9-0fe87de4ddc8"
-			"3c9f767e-7a42-4dd9-935c-237c9c5c47e9" "3ea086ab-6a6b-401a-84f1-665853ca4a09"
-			"461b6d80-51ed-45b7-b191-498d2b17c8e0" "49c4b093-6a01-41fb-9f81-6b8baae5c120"
-			"4c18506e-7ebe-457b-95e9-b9c30a62c7e8" "4dddb44c-9edf-4fbf-93e7-a8117b2d3ff9"
-			"50d831af-fc12-4807-8dca-ed14686d1643" "5367c6a8-7831-4841-a983-0918578c43d5"
-			"5af03697-723d-4b26-af65-042ede7503bb" "5c6fc10e-efea-45de-8f12-d340decd9cde"
-			"649a82e5-7220-4f44-977d-78f3cb5ec726" "64e7e232-ac41-4039-842f-dfa5f3af96de"
-			"69c7a140-cd95-4f51-8947-e9f4feee331e" "742e4432-2949-450c-9d19-0121adec59c6"
-			"7708ba6d-058d-4bff-bda7-2cc83358d7b8" "77812977-850d-4ddf-a66a-e14004ab5c7d"
-			"7866eed2-597e-485b-8956-f936717947e0" "787b9d29-60bf-498b-a3fa-4704e40668b2"
-			"88733451-aa05-465d-aa4b-dc85c4c290db" "892b4ab3-1517-4362-8394-104e91cb9425"
-			"8f91a66f-67cc-4066-b1fb-960c65d33439" "948a029b-d7a3-40ad-81bd-1d10d56fd6e8"
-			"960a5c3a-5104-4712-bd1c-74295566bb0b" "98aa87e7-8994-4938-a240-386e91d93a3a"
-			"9b05f0c6-f2ba-4198-9307-af848d04a704" "a3583de0-e791-47df-8599-1bcfe1215194"
-			"a4d5f4cd-5351-4dc7-889c-3ea2c2bb94a3" "af9a3320-e2b0-41e5-b494-50bd447c4e7d"
-			"b1841387-03fa-4da1-bb23-7ea818e6dc41" "b31ed106-d5a7-4352-85ab-aadf9a960c65"
-			"b3f57591-6e5a-4b19-8b1b-68ccbd40f49c" "b6d03dff-32eb-4125-be5e-3e0aeeb1e988"
-			"b706acc0-7d3a-43bf-b453-0f4fb704f922" "b71288df-952b-4256-b756-b4fe12eede31"
-			"b852a435-3038-4391-9935-f5d804f0c3d9" "b8f8ba5f-4cc9-47bd-87ff-e60b9c1974a0"
-			"bd93e0ff-270a-48e3-a5f7-b2889a67adf7" "cec91af8-9061-4f23-baf9-c422045edbe5"
-			"d15abc3a-76b6-4117-89db-c94f32e11855" "d282ec32-64c6-42f6-be5e-4b299fd2d07c"
-			"d45b25c6-faf6-4bcf-8f4e-2af9ab2e4add" "d744ed62-1993-41c7-8b4b-5aa56a5ab411"
-			"d7bebb15-180d-40a8-850e-0ba244dc3c0f" "d8ac9060-796c-42f1-9bbc-27becbf0348d"
-			"d9f30ea8-18d3-4348-9390-5ecdb03d50d1" "dba2d7a6-ba97-42be-8454-bb7d5edbd110"
-			"dbcd88db-5423-4ff2-8ed8-c2035994e527" "e19ba480-294d-421f-9869-e83b6455b51e"
-			"e38d4dd4-c357-46b7-be9c-e9d71cc3aa05" "e793ad08-1bb3-49c5-916b-81c26f60eb2c"
-			"e7bf13c1-bd70-4ff1-b532-305068298e52" "eb2d36fe-dec6-47f8-90ec-e4ef6b9d53ed"
+			"189e168f-b7a0-484c-aa2a-fdb9d9e916c6" "1feb841d-fd24-4e8e-b5aa-f776dbc4f00d"
+			"20235f43-cf96-4218-aa84-5a156a011ff2" "26c525f2-d4d9-4653-8977-4d813e08275d"
+			"29dd66b1-5e01-40b9-8e29-19c8a0c273a8" "2c4f203c-5b0c-4867-8517-6ca5922d05ff"
+			"2cb49122-9564-4c5b-856a-4b720769080a" "301259ed-6e02-41d2-bbbf-7d9d5a8ac4dd"
+			"3c5fac19-14d4-4494-9de9-0fe87de4ddc8" "3c9f767e-7a42-4dd9-935c-237c9c5c47e9"
+			"3ea086ab-6a6b-401a-84f1-665853ca4a09" "461b6d80-51ed-45b7-b191-498d2b17c8e0"
+			"49c4b093-6a01-41fb-9f81-6b8baae5c120" "4c18506e-7ebe-457b-95e9-b9c30a62c7e8"
+			"4c61aa9c-b6b6-4ffb-9696-fa037898494f" "4dddb44c-9edf-4fbf-93e7-a8117b2d3ff9"
+			"50d831af-fc12-4807-8dca-ed14686d1643" "526dd3a9-6bc9-4151-9490-1382553dbada"
+			"5367c6a8-7831-4841-a983-0918578c43d5" "5af03697-723d-4b26-af65-042ede7503bb"
+			"5c6fc10e-efea-45de-8f12-d340decd9cde" "649a82e5-7220-4f44-977d-78f3cb5ec726"
+			"64e7e232-ac41-4039-842f-dfa5f3af96de" "69c7a140-cd95-4f51-8947-e9f4feee331e"
+			"742e4432-2949-450c-9d19-0121adec59c6" "7708ba6d-058d-4bff-bda7-2cc83358d7b8"
+			"77812977-850d-4ddf-a66a-e14004ab5c7d" "7866eed2-597e-485b-8956-f936717947e0"
+			"787b9d29-60bf-498b-a3fa-4704e40668b2" "88733451-aa05-465d-aa4b-dc85c4c290db"
+			"892b4ab3-1517-4362-8394-104e91cb9425" "8f91a66f-67cc-4066-b1fb-960c65d33439"
+			"948a029b-d7a3-40ad-81bd-1d10d56fd6e8" "960a5c3a-5104-4712-bd1c-74295566bb0b"
+			"98aa87e7-8994-4938-a240-386e91d93a3a" "9b05f0c6-f2ba-4198-9307-af848d04a704"
+			"a3583de0-e791-47df-8599-1bcfe1215194" "a4d5f4cd-5351-4dc7-889c-3ea2c2bb94a3"
+			"af9a3320-e2b0-41e5-b494-50bd447c4e7d" "b1841387-03fa-4da1-bb23-7ea818e6dc41"
+			"b31ed106-d5a7-4352-85ab-aadf9a960c65" "b3f57591-6e5a-4b19-8b1b-68ccbd40f49c"
+			"b6d03dff-32eb-4125-be5e-3e0aeeb1e988" "b706acc0-7d3a-43bf-b453-0f4fb704f922"
+			"b71288df-952b-4256-b756-b4fe12eede31" "b852a435-3038-4391-9935-f5d804f0c3d9"
+			"b8f8ba5f-4cc9-47bd-87ff-e60b9c1974a0" "bd93e0ff-270a-48e3-a5f7-b2889a67adf7"
+			"cec91af8-9061-4f23-baf9-c422045edbe5" "d15abc3a-76b6-4117-89db-c94f32e11855"
+			"d282ec32-64c6-42f6-be5e-4b299fd2d07c" "d45b25c6-faf6-4bcf-8f4e-2af9ab2e4add"
+			"d744ed62-1993-41c7-8b4b-5aa56a5ab411" "d7bebb15-180d-40a8-850e-0ba244dc3c0f"
+			"d8ac9060-796c-42f1-9bbc-27becbf0348d" "d9f30ea8-18d3-4348-9390-5ecdb03d50d1"
+			"dba2d7a6-ba97-42be-8454-bb7d5edbd110" "dbcd88db-5423-4ff2-8ed8-c2035994e527"
+			"e19ba480-294d-421f-9869-e83b6455b51e" "e38d4dd4-c357-46b7-be9c-e9d71cc3aa05"
+			"e793ad08-1bb3-49c5-916b-81c26f60eb2c" "e7bf13c1-bd70-4ff1-b532-305068298e52"
+			"e7d7e490-93c0-4022-827f-f329053ecd3d" "eb2d36fe-dec6-47f8-90ec-e4ef6b9d53ed"
 			"f269a27b-9eea-4bed-8032-1cbdef2252f6" "f6f4338e-928d-4394-a0c8-883e8343ab37"
 			"f8e644cc-d25f-4029-8395-1f56e1c81958" "fd81428f-132e-4115-b826-9852979ae8ee"
